File: hardware/avionics/avionics_dev_board/avionics_dev_board.kicad_pcb (KiCad board)
At the start: 4 copper layers, 91.5 x 78.9 mm, 103 parts, among them J1-MCU Conn_01x02, J2-ACC Conn_01x02, J4-PMAG Conn_01x02, J6-M10S Conn_01x02, J7-W25Q Conn_01x02, J8-L62 Conn_01x02, J9-L80 Conn_01x02, M10S MAX-M10S-00B, Q3 FDS2734, T1-MBAT Main battery, T2-PBAT Parachute battery, T3-NICH Nichrome connector, Y1 16MHz

Commit message: Added power isolation jumper to regulator output and improved fuse placement
Parts:
- added J1-3V3: Conn_01x02, Connector_PinHeader_2.54mm:PinHeader_1x02_P2.54mm_Vertical, F.Cu at (202.2, 34.0)
- moved PWR_SW 8.18 mm to (187.7, 48.9)
- moved F1 3.85 mm to (192.2, 44.9)
- moved C3 1.77 mm to (197.4, 40.8)
- moved C9 1.77 mm to (196.4, 33.8)
- moved L1 1.77 mm to (196.4, 38.0)
- moved R1 1.77 mm to (205.4, 40.0)
- moved BUCK 1.77 mm to (201.3, 39.1)
- moved C4 1.77 mm to (206.6, 37.4)
- moved C7 1.77 mm to (198.2, 38.2)
- moved C8 1.77 mm to (198.6, 33.8)
- moved PWR_LED 1.77 mm to (195.0, 31.0)
- moved R2 1.77 mm to (204.6, 37.4)
- moved R3 1.77 mm to (194.2, 33.8)
- moved C2 1.77 mm to (198.6, 43.8)
- moved D2 1.77 mm to (196.3, 44.3)
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- renumbered J1-MCU to J2-MCU, J2-ACC to J3-ACC, RST1 to RST
Connections:
- C1 pad 2: Net-(PWR_SW1-A) -> Net-(D2-A)
- C4 pad 1: +3V3 -> /BUCK_OUT
- C8 pad 2: +3V3 -> /BUCK_OUT
- C9 pad 2: +3V3 -> /BUCK_OUT
- L1 pad 2: +3V3 -> /BUCK_OUT
- R2 pad 2: +3V3 -> /BUCK_OUT
- R3 pad 1: +3V3 -> /BUCK_OUT
Routing:
- net +3V3: track 40.9 -> 16.3 mm, vias 15 -> 8
- net /BUCK_OUT: track 0.00 -> 16.6 mm
- net Net-(PWR_SW1-B): track 27.8 -> 17.4 mm
- net Net-(PWR_SW1-A): track 10.2 -> 4.51 mm
- net Net-(D2-A): track 2.40 -> 4.15 mm
- net GND: track 150.6 -> 149.7 mm
Other:
- board text added: "."

Commit message: Devlog update
Parts:
- F1: footprint Fuse:Fuse_0603_1608Metric -> Fuse:Fuse_1206_3216Metric
- PWR_LED, ULED: footprint LED_SMD:LED_0603_1608Metric -> LED_SMD:LED_0805_2012Metric
- moved PWR_SW 0.60 mm to (187.1, 48.9)
- moved F1 0.30 mm to (191.9, 44.9)
- moved ULED 0.20 mm to (172.9, 95.3)
- moved PWR_LED 0.19 mm to (195.0, 30.8)
Routing:
- net Net-(D2-A): track 4.15 -> 4.76 mm
