File: hardware/avionics/avionics_dev_board/avionics_dev_board.kicad_sch (KiCad schematic)
At the start: 93 parts, among them J1-MBAT1 Main battery, J10-PBAT1 Parachute battery, J9-NICH1 Nichrome connector, M10S1 MAX-M10S-00B, Q3 FDS2734, Y1 16MHz

Commit message: Improved shielding of GPS RF trace and added 0 ohm resistors to switch SWD RX and TX if necessary
Parts:
- removed TP1, TP10, TP11, TP2, TP3, TP4, TP5, TP6, TP7, TP8, TP9: TestPoint, TestPoint:TestPoint_Pad_D1.0mm, symbol Connector:TestPoint
- added R10, R5, R6, R9: 0R, Resistor_SMD:R_0603_1608Metric, symbol Device:R
- C20, C21: value 10pF -> 12pF
Connections:
- net VCP_RX: now also MCU1.33 (PB11), R5.2, R9.1; no longer MCU1.30 (PB10), SWD_INT1.13 (Pin_13)
- net VCP_TX: now also MCU1.30 (PB10), R10.2, R6.2; no longer MCU1.33 (PB11), SWD_INT1.14 (Pin_14)
- new net: R6.1, R9.2, SWD_INT1.14 (Pin_14)
- new net: R10.1, R5.1, SWD_INT1.13 (Pin_13)
Other:
- note added: "Duplicate 0 ohm resistors incase RX-TX pair swapped"
- moved on the sheet: C37, J10-PBAT1, J9-NICH1, PARA_ARM1, Q3, R11, R12

Commit message: Added pull up/down resistors to some pins according to datasheet recommendations
Parts:
- added R16, R17, R18: 10kR, Resistor_SMD:R_0603_1608Metric, symbol Device:R
Connections:
- net +3V3: now also R17.2, R18.2; no longer W25Q1.3 (DO_(IO1)_2)
- net CS_W25Q: now also R17.1
- net GND: now also R16.1
- net LSM6_INT1: now also R16.2
- net NRST: now also R18.1
- net at BUCK1.3 (VIN), BUCK1.5 (EN), C3.2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: now also C2.2
- net at D2.2 (A), F1.2: no longer C2.2
- net WP_W25Q: now reaches MCU1.39 (PC7)
- net WP_W25Q: now also W25Q1.3 (DO_(IO1)_2)
- net RST_W25Q renamed HOLD_W25Q
- no-connect marks 35 -> 34
Other:
- moved on the sheet: C10, C11, C12, C15, C16, C17, C19, C2, C23, C24, C33, C5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

Commit message: Log file update
Parts:
- BUCK1: value TPS563200 -> TPS563208
- SWD_INT1: footprint Connector_PinHeader_2.54mm:PinHeader_2x07_P2.54mm_Vertical -> Connector_PinSocket_1.27mm:PinSocket_2x07_P1.27mm_Vertical
Other:
- moved on the sheet: C36, R10, R5, R6, R9, SWD_INT1

Commit message: Avionics dev board V2
Parts:
- added C38: 100nF, Capacitor_SMD:C_0603_1608Metric, symbol Device:C
- added J1-MCU1, J2-ACC1, J4-PMAG1, J6-M10S1, J7-W25Q1, J8-L62, J9-L80: Conn_01x02, Connector_PinHeader_2.54mm:PinHeader_1x02_P2.54mm_Vertical, symbol Connector_Generic:Conn_01x02
- added R19: 10kR, Resistor_SMD:R_0603_1608Metric, symbol Device:R
- added R20: 220R, Resistor_SMD:R_0603_1608Metric, symbol Device:R
- added TP-3V3, TP-GND1: TestPoint, TestPoint:TestPoint_Pad_D1.0mm, symbol Connector:TestPoint
- added UBT1: SW_Push, avionicsw:hanxia HX 3x4x2-2P-1.6N TACTILE SWITCH, symbol Switch:SW_Push
- added ULED2: PWR LED, LED_SMD:LED_0603_1608Metric, symbol Device:LED
- R3: value 1kR -> 220R
- RST1: footprint avionicsw:G-Switch GT-TC060A-H025-L1S -> avionicsw:hanxia HX 3x4x2-2P-1.6N TACTILE SWITCH
- renumbered J1-MBAT1 to T1-MBAT1, J10-PBAT1 to T2-PBAT1, J9-NICH1 to T3-NICH1
Connections:
- net +3V3: now also J1-MCU1.2 (Pin_2), J2-ACC1.2 (Pin_2), J4-PMAG1.2 (Pin_2), J6-M10S1.1 (Pin_1), J7-W25Q1.2 (Pin_2), J8-L62.1 (Pin_1), J9-L80.1 (Pin_1), R19.2, TP-3V3.1; no longer ADXL1.1 (VDD_I/O), ADXL1.6 (VS), BMP1.1 (VDDIO), BMP1.10 (VDD), BMP1.6 (CSB), C10.1, C11.1, C12.1, C13.1, C17.1, C23.2, C24.2, C25.2, C26.2, C27.2, C28.2, C30.2, C31.2, C32.2, C33.2, C34.2, C35.2, C5.1, C6.1, FB1.2, L62-1.3 (Pin_3), L80-1.3 (Pin_3), LSM6.P$5 (VDDIO), LSM6.P$8 (VDD), M10S1.7 (V_IO), M10S1.8 (VCC), MCU1.1 (VBAT), MCU1.16 (VDD), MCU1.32 (VDD), MCU1.48 (VDD), MCU1.64 (VDD), MMC1.13 (VDDIO), MMC1.2 (VDD), MMC1.4 (~{SPI_CS}), R17.2, R7.2, R8.2, W25Q1.8 (VCC)
- net GND: now also C38.2, TP-GND1.1, UBT1.1, ULED2.1 (K)
- net at MCU1.40 (PC8): now also C38.1, R19.1, UBT1.2
- net at MCU1.41 (PC9): now also R20.2
- new net: R20.1, ULED2.2 (A)
- new net L62_VCC: C34.2, J8-L62.2 (Pin_2), L62-1.3 (Pin_3)
- new net L80_VCC: C35.2, J9-L80.2 (Pin_2), L80-1.3 (Pin_3)
- new net VCC-ACC: ADXL1.1 (VDD_I/O), ADXL1.6 (VS), C23.2, C24.2, C25.2, C26.2, J2-ACC1.1 (Pin_1), LSM6.P$5 (VDDIO), LSM6.P$8 (VDD)
- new net VCC-M10S: C31.2, C32.2, J6-M10S1.2 (Pin_2), M10S1.7 (V_IO), M10S1.8 (VCC)
- new net VCC-MCU: C10.1, C11.1, C12.1, C13.1, C17.1, C5.1, C6.1, FB1.2, J1-MCU1.1 (Pin_1), MCU1.1 (VBAT), MCU1.16 (VDD), MCU1.32 (VDD), MCU1.48 (VDD), MCU1.64 (VDD)
- new net VCC-PMAG: BMP1.1 (VDDIO), BMP1.10 (VDD), BMP1.6 (CSB), C27.2, C28.2, C30.2, J4-PMAG1.1 (Pin_1), MMC1.13 (VDDIO), MMC1.2 (VDD), MMC1.4 (~{SPI_CS}), R7.2, R8.2
- new net VCC-W25Q: C33.2, J7-W25Q1.1 (Pin_1), R17.2, W25Q1.8 (VCC)
- no-connect marks 34 -> 32
Other:
- moved on the sheet: AE1, ANT_24, ANT_868, C31, C32, C33, C34, C35, C36, C37, L62-1, L62-2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

Commit message: Added power isolation jumper to regulator output and improved fuse placement
Parts:
- added J1-3V3: Conn_01x02, Connector_PinHeader_2.54mm:PinHeader_1x02_P2.54mm_Vertical, symbol Connector_Generic:Conn_01x02
- renumbered J1-MCU1 to J2-MCU1, J2-ACC1 to J3-ACC1
Connections:
- net +3V3: now also J1-3V3.2 (Pin_2); no longer C4.1, C8.2, C9.2, L1.2, R2.2, R3.1
- net at F1.1, PWR_SW1.1 (A): no longer C1.2
- net at D2.2 (A), F1.2: now also C1.2
- new net BUCK_OUT: C4.1, C8.2, C9.2, J1-3V3.1 (Pin_1), L1.2, R2.2, R3.1
Other:
- moved on the sheet: C1, F1

Commit message: Devlog update
Parts:
- F1: footprint Fuse:Fuse_0603_1608Metric -> Fuse:Fuse_1206_3216Metric
- PWR_LED1, ULED2: footprint LED_SMD:LED_0603_1608Metric -> LED_SMD:LED_0805_2012Metric
Changed lines of the file:
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@@
 			)
 		)
-		(property "Footprint" "LED_SMD:LED_0603_1608Metric"
+		(property "Footprint" "LED_SMD:LED_0805_2012Metric"
 			(at 561.34 443.23 0)
 			(effects
@@
 			)
 		)
-		(property "Footprint" "LED_SMD:LED_0603_1608Metric"
+		(property "Footprint" "LED_SMD:LED_0805_2012Metric"
 			(at 433.07 365.76 0)
 			(effects
@@
 			)
 		)
-		(property "Footprint" "Fuse:Fuse_0603_1608Metric"
+		(property "Footprint" "Fuse:Fuse_1206_3216Metric"
 			(at 322.58 351.028 90)
 			(effects
