File: hardware/ground_station/rf_controller/rf_controller.kicad_pcb (KiCad board)
At the start: 4 copper layers, 0 parts

Commit message: PCB layout for RF controller And additional updates to schematic: - Added ESD protection to USB data lines - Fixed wrong placement of capacitors around LDO voltage regulator - Added extra user LED and button
Parts:
- added ANT_24: 2.4GHz antenna, Connector_Coaxial:SMA_Amphenol_901-144_Vertical, F.Cu at (583.2, 313.6)
- added ANT_868: 868MHz antenna, Connector_Coaxial:SMA_Amphenol_901-144_Vertical, F.Cu at (624.1, 306.6)
- added BOOT_SW1: SW_SPDT, avionicsw:SHOU HAN SS12D10G5, F.Cu at (583.5, 350.4)
- added C1: 100nF, Capacitor_SMD:C_0603_1608Metric, F.Cu at (586.8, 366.6)
- added C10: 100nF, Capacitor_SMD:C_0603_1608Metric, F.Cu at (615.6, 355.3)
- added C11: 100nF, Capacitor_SMD:C_0603_1608Metric, F.Cu at (600.4, 355.2)
- added C12: 100nF, Capacitor_SMD:C_0603_1608Metric, F.Cu at (603.2, 353.1)
- added C13: 1uF, Capacitor_SMD:C_0603_1608Metric, F.Cu at (613.6, 371.7)
- added C14: 10nF, Capacitor_SMD:C_0603_1608Metric, F.Cu at (610.2, 368.4)
- added C15: 100nF, Capacitor_SMD:C_0603_1608Metric, F.Cu at (610.2, 370.1)
- added C16: 1uF, Capacitor_SMD:C_0603_1608Metric, F.Cu at (610.2, 371.8)
- added C17: 100nF, Capacitor_SMD:C_0603_1608Metric, F.Cu at (601.5, 365.7)
- added C18: 1uF, Capacitor_SMD:C_0603_1608Metric, F.Cu at (610.2, 373.5)
- added C19: 100nF, Capacitor_SMD:C_0603_1608Metric, F.Cu at (593.6, 352.0)
- added C20: 12pF, Capacitor_SMD:C_0603_1608Metric, F.Cu at (596.0, 359.0)
- added C21: 12pF, Capacitor_SMD:C_0603_1608Metric, F.Cu at (598.9, 362.2)
- added C22: 100nF, Capacitor_SMD:C_0603_1608Metric, F.Cu at (605.8, 351.1)
- added C23: 22uF, Capacitor_SMD:C_0805_2012Metric, F.Cu at (625.3, 339.5)
- added C24: 1uF, Capacitor_SMD:C_0805_2012Metric, F.Cu at (627.7, 339.5)
- added C25: 1uF, Capacitor_SMD:C_0805_2012Metric, F.Cu at (623.3, 350.7)
- added C34: 100nF, Capacitor_SMD:C_0603_1608Metric, F.Cu at (620.3, 312.3)
- added C35: 100nF, Capacitor_SMD:C_0603_1608Metric, F.Cu at (578.0, 325.1)
- added C36: 100nF, Capacitor_SMD:C_0603_1608Metric, F.Cu at (588.0, 364.0)
- added C38: 100nF, Capacitor_SMD:C_0603_1608Metric, F.Cu at (623.2, 369.8)
- added C5: 100nF, Capacitor_SMD:C_0603_1608Metric, F.Cu at (613.7, 367.6)
- added C6: 4u7F, Capacitor_SMD:C_0805_2012Metric, F.Cu at (600.2, 353.0)
- added F2: 500mA, Fuse:Fuse_1206_3216Metric, F.Cu at (621.4, 338.5)
- added FB1: 120R, Inductor_SMD:L_0603_1608Metric, F.Cu at (613.6, 373.5)
- added H1: MountingHole, MountingHole:MountingHole_2.2mm_M2, F.Cu at (510.6, 296.2)
- added H2: MountingHole, MountingHole:MountingHole_2.2mm_M2, F.Cu at (509.8, 305.2)
- added H3: MountingHole, MountingHole:MountingHole_2.2mm_M2, F.Cu at (509.8, 311.1)
- added H4: MountingHole, MountingHole:MountingHole_2.2mm_M2, F.Cu at (509.8, 317.1)
- added J1: USB_C_Receptacle_USB2.0_16P, Connector_USB:USB_C_Receptacle_G-Switch_GT-USB-7010ASV, F.Cu at (627.8, 358.1)
- added J1-3V3: Conn_01x02, Connector_PinHeader_2.54mm:PinHeader_1x02_P2.54mm_Vertical, F.Cu at (621.1, 346.7)
- added J2-MCU1: Conn_01x02, Connector_PinHeader_2.54mm:PinHeader_1x02_P2.54mm_Vertical, F.Cu at (597.3, 368.2)
- added J8-L62: Conn_01x02, Connector_PinHeader_2.54mm:PinHeader_1x02_P2.54mm_Vertical, F.Cu at (598.0, 315.7)
- added J9-L80: Conn_01x02, Connector_PinHeader_2.54mm:PinHeader_1x02_P2.54mm_Vertical, F.Cu at (592.6, 313.1)
- added L62-1: LAMBDA62, Connector_PinSocket_2.54mm:PinSocket_1x08_P2.54mm_Vertical, F.Cu at (624.1, 315.2)
- added L62-2: Conn_01x08_Socket, Connector_PinSocket_2.54mm:PinSocket_1x08_P2.54mm_Vertical, F.Cu at (606.3, 332.0)
- added L80-1: LAMBDA80, Connector_PinSocket_2.54mm:PinSocket_1x08_P2.54mm_Vertical, F.Cu at (580.9, 321.3)
- added L80-2: Conn_01x08_Socket, Connector_PinSocket_2.54mm:PinSocket_1x08_P2.54mm_Vertical, F.Cu at (597.7, 339.1)
- added MCU1: STM32G474RET6, Package_QFP:LQFP-64_10x10mm_P0.5mm, F.Cu at (608.5, 360.6)
- added PWR_LED2: PWR LED, LED_SMD:LED_0805_2012Metric, F.Cu at (627.7, 350.7)
- added PWR_SW2: SW_SPDT, avionicsw:SHOU HAN SS12D10G5, F.Cu at (614.9, 343.9)
- added R1: 5k1R, Resistor_SMD:R_0603_1608Metric, F.Cu at (620.5, 361.5)
- added R18: 10kR, Resistor_SMD:R_0603_1608Metric, F.Cu at (590.2, 355.9)
- added R19: 10kR, Resistor_SMD:R_0603_1608Metric, F.Cu at (619.1, 366.3)
- added R2: 5k1R, Resistor_SMD:R_0603_1608Metric, F.Cu at (620.5, 354.8)
- added R20: 220R, Resistor_SMD:R_0603_1608Metric, F.Cu at (628.6, 366.3)
- added R3: 10kR, Resistor_SMD:R_0603_1608Metric, F.Cu at (591.0, 369.8)
- added R4: 10kR, Resistor_SMD:R_0603_1608Metric, F.Cu at (605.8, 352.8)
- added R5: 220R, Resistor_SMD:R_0603_1608Metric, F.Cu at (603.5, 368.6)
- added R6: 220R, Resistor_SMD:R_0603_1608Metric, F.Cu at (625.6, 350.7)
- added RST1: SW_Push, avionicsw:hanxia HX 3x4x2-2P-1.6N TACTILE SWITCH, F.Cu at (591.0, 352.0)
- added SWD_INT1: SWD interface, Connector_PinSocket_1.27mm:PinSocket_2x07_P1.27mm_Vertical, F.Cu at (589.8, 361.6)
- added TP-3V3: TestPoint, TestPoint:TestPoint_Pad_D1.0mm, F.Cu at (592.6, 308.8)
- added TP-GND1: TestPoint, TestPoint:TestPoint_Pad_D1.0mm, F.Cu at (599.0, 308.8)
- added U1: LDL112PV33R, LDL112PV33R:DFN_2PV33R_STM, F.Cu at (621.9, 342.3)
- added U3: USBLC6-2SC6, Package_TO_SOT_SMD:SOT-23-6, F.Cu at (619.2, 358.1)
- added UBT1: SW_Push, avionicsw:hanxia HX 3x4x2-2P-1.6N TACTILE SWITCH, F.Cu at (623.1, 367.2)
- added UBT2: SW_Push, avionicsw:hanxia HX 3x4x2-2P-1.6N TACTILE SWITCH, F.Cu at (586.8, 369.2)
- added ULED1: PWR LED, LED_SMD:LED_0805_2012Metric, F.Cu at (628.6, 368.3)
- added ULED2: PWR LED, LED_SMD:LED_0805_2012Metric, F.Cu at (603.6, 370.5)
- added Y1: 16MHz, ABM8G-16.000MHZ-4Y-T3:XTAL_ABM8G-16.000MHZ-4Y-T3, F.Cu at (598.9, 359.0)
Routing:
- net GND: track 0.00 -> 105.6 mm, vias 0 -> 97
- net /L62_RXSW: track 0.00 -> 72.1 mm, vias 0 -> 1
- net /L62_BUSY: track 0.00 -> 66.9 mm, vias 0 -> 2
- net /L62_TXSW: track 0.00 -> 58.7 mm, vias 0 -> 3
- net /SPI3_MOSI: track 0.00 -> 58.7 mm, vias 0 -> 1
- net /L62_DIO1: track 0.00 -> 57.4 mm
- net /VCP_RX: track 0.00 -> 55.4 mm
- net /SPI3_MISO: track 0.00 -> 51.3 mm, vias 0 -> 1
- net /VCP_TX: track 0.00 -> 50.8 mm, vias 0 -> 1
- net /L62_DIO2: track 0.00 -> 50.2 mm, vias 0 -> 1
- net /SPI3_SCK: track 0.00 -> 45.3 mm
- net /L80_DIO3: track 0.00 -> 43.8 mm, vias 0 -> 1
- net /L80_BUSY: track 0.00 -> 41.4 mm, vias 0 -> 2
- net /L80_CS: track 0.00 -> 40.7 mm
- net /L80_DIO2: track 0.00 -> 40.5 mm, vias 0 -> 2
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- added copper zone on In2.Cu, net +3V3
- added copper zone on In2.Cu, net /VCC-MCU
- added copper zone on B.Cu, net GND
- added copper zone on F.Cu, net GND
- added copper zone on In1.Cu, net GND
- added copper zone on In2.Cu, net GND
Other:
- board outline added: 54.9 x 73.6 mm

Commit message: Finalised RF controller PCB layout
Parts:
- removed H4: MountingHole, MountingHole:MountingHole_2.2mm_M2
- moved H2 137.2 mm to (628.9, 373.2)
- moved H1 102.9 mm to (578.8, 373.2)
- moved H3 94.4 mm to (603.9, 304.2)
- moved J8-L62 14.7 mm to (611.0, 308.9), turned to 90 degrees
- moved TP-3V3 13.2 mm to (605.7, 307.4)
- moved TP-GND 6.91 mm to (605.7, 310.5)
- moved ANT_24 5.35 mm to (583.2, 308.2)
- moved J9-L80 2.69 mm to (594.6, 311.4), turned to -90 degrees
- renumbered BOOT_SW1 to BOOT_SW, J2-MCU1 to J2-MCU, MCU1 to MCU, PWR_LED2 to PWR_LED, PWR_SW2 to PWR_SW, RST1 to RST, SWD_INT1 to SWD_INT, TP-GND1 to TP-GND
Routing:
- net /L62_VCC: track 25.0 -> 10.4 mm
- net /L80_ANT: track 8.70 -> 14.1 mm
- net /L80_VCC: track 19.3 -> 22.8 mm
- net +3V3: track 12.7 -> 14.3 mm
- net /BOOT0: track 40.1 -> 39.0 mm
- net /L62_BUSY: track 66.9 -> 67.9 mm
- net /SWO: track 26.0 -> 26.9 mm
- net /L62_CS: track 30.9 -> 31.7 mm
- net /L62_RST: track 35.5 -> 34.8 mm
- net /L80_DIO2: track 40.5 -> 39.8 mm
- net /L62_DIO2: track 50.2 -> 50.7 mm
- net GND: track 105.6 -> 105.5 mm, vias 97 -> 104
- net /L62_TXSW: vias 3 -> 1
- net (no net): vias 4 -> 0
Other:
- board size 54.9 x 73.6 mm -> 55.7 x 74.1 mm
